File: Eagle/Current Owl files/double_layer.brd (EAGLE design)
At the start: 68.6 x 47 mm, 21 parts, among them J1 2X6 FEMALE, J2 2X6 FEMALE, Q1 2N3906, X1 SMA-142-0701-851/861

Commit message: updated eagle files
Parts:
- removed X1: SMA-142-0701-851/861, con-coax:J502-ND-142-0701-851/861
- added J$1: SMA_EDGE, SparkFun-Retired:SMA-EDGE
- moved J12 29.2 mm to (7.62, 20.3)
- moved J7 19.9 mm to (25.4, 21.6)
- moved J4 8.13 mm to (19.1, 2.54)
- moved J5 5.08 mm to (29.2, 2.54)
- moved Q1 1.27 mm to (21.6, 7.62), turned to 180 degrees
Connections:
- removed net N$3: LS1.-, Q1.3
- new net N$1: LS1.-, Q1.1
- net GND: now also J$1.GND@0, J$1.GND@1, J$1.GND@2, J$1.GND@3; no longer X1.G@1, X1.G@2, X1.G@3, X1.G@4
- net N$8: now also J$1.SIG; no longer X1.1
- net RAW: now also Q1.3; no longer Q1.1
Routing:
- net GND: track 178.3 -> 147.2 mm, vias 3 -> 4
- net N$11: track 8.89 -> 19.9 mm
- net N$3: track 9.42 -> 0.00 mm
- net N$2: track 9.20 -> 0.00 mm
- net N$1: track 0.00 -> 8.89 mm
- net N$10: track 5.08 -> 12.5 mm
- net RAW: track 35.1 -> 42.2 mm
- net N$6: track 24.7 -> 22.2 mm
- net N$5: track 1.80 -> 0.00 mm
- net N$4: track 1.80 -> 0.00 mm
- net VCC: track 102.5 -> 103.2 mm
