File: Eagle/Current Owl files/schematic02.brd (EAGLE design)
At the start: 68.6 x 49.5 mm, 23 parts, among them J1 2X6 FEMALE, J2 2X6 FEMALE, Q1 2N3906, X1 SMA-142-0701-851/861

Commit message: updated eagle files
Parts:
- removed J13: (no value), SparkFun-Connectors:JST-3-PTH
- removed J14: (no value), SparkFun-Connectors:1X02
- removed R2: 10k, SparkFun-Resistors:AXIAL-0.3
- added GPSCONN: (no value), SparkFun-Connectors:1X03
- moved X1 7.62 mm to (-1.27, 29.2)
- moved J6 5.24 mm to (7.62, 16.5)
- moved Q1 5.24 mm to (22.9, 7.62)
- moved J7 5.08 mm to (2.54, 16.5)
- moved LS1 2.54 mm to (16.5, 16.5)
- moved BTN 2.54 mm to (59.7, 29.2)
- moved S_ANT 1.80 mm to (6.35, 31.8)
- moved ANT_EXT 1.27 mm to (6.35, 40.6)
- moved J9 1.27 mm to (11.4, 44.5)
Connections:
- removed net N$6: R2.P$2, S_MODE.2
- removed net N$9: J14.2
- net 7: now also S_MODE.2; no longer R2.P$1
- net 8: now also GPSCONN.3
- net GND: now also GPSCONN.2; no longer J13.2, J14.1, Q1.3
- net N$3: now also Q1.3; no longer Q1.1
- net RAW: now also Q1.1
- net VCC: now also GPSCONN.1; no longer J13.1
Routing:
- net GND: track 188.8 -> 1.80 mm, vias 4 -> 0
- net N$9: track 19.9 -> 0.00 mm
- net 7: track 3.81 -> 11.5 mm
- net N$6: track 5.61 -> 0.00 mm
- net N$8: track 9.94 -> 5.08 mm
- net N$1: track 29.3 -> 24.7 mm
- net VCC: track 104.0 -> 100.2 mm
- net RAW: track 29.8 -> 27.2 mm
- net N$3: track 11.7 -> 9.42 mm
- net N$7: track 5.08 -> 6.35 mm
- net 10: track 4.58 -> 3.81 mm
- net ANT: track 12.5 -> 13.0 mm
- net 8: vias 1 -> 0
- added copper zone on layer 16, net GND
- removed copper zone on layer 1, net GND
Other:
- board size 68.6 x 49.5 mm -> 68.6 x 47 mm
