File: Eagle/Current Owl files/schematic02.sch (EAGLE design)
At the start: 22 parts, among them J1 2X6 FEMALE, J2 2X6 FEMALE, Q1 2N3906, X1 SMA-142-0701-851/861

Commit message: updated eagle files
Parts:
- removed J13: (no value), SparkFun-Connectors:CONN_03JST-PTH
- removed J14: (no value), SparkFun-Connectors:CONN_02
- added GPSCONN: (no value), SparkFun-Connectors:CONN_03
Connections:
- net N$6 renamed 7
- removed net N$9: J14.2
- net 8: now also GPSCONN.3
- net GND: now also GPSCONN.2; no longer J13.2, J14.1, Q1.E
- net N$3: now also Q1.E; no longer Q1.C
- net RAW: now also Q1.C
- net VCC: now also GPSCONN.1; no longer J13.1
Other:
- moved on the sheet: Q1
Changed lines of the file:
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@@
 <?xml version="1.0" encoding="utf-8"?>
 <!DOCTYPE eagle SYSTEM "eagle.dtd">
-<eagle version="8.1.0">
+<eagle version="6.5.0">
 <drawing>
 <settings>
@@
 <part name="J2" library="SparkFun-Connectors" deviceset="CONN_06X2" device="PTH_FEMALE" value="2X6 FEMALE"/>
 <part name="S_MODE" library="SparkFun-Switches" deviceset="SWITCH-SPDT" device="-PTH-11.6X4.0MM"/>
+<part name="GPSCONN" library="SparkFun-Connectors" deviceset="CONN_03" device=""/>
 <part name="X1" library="con-coax" deviceset="SMA-" device="142-0701-851/861"/>
 <part name="LS1" library="SparkFun-Electromechanical" deviceset="BUZZER" device="-PTH"/>
@@
 <part name="J11" library="SparkFun-Connectors" deviceset="CONN_12" device=""/>
 <part name="J12" library="SparkFun-Connectors" deviceset="CONN_01" device=""/>
-<part name="J13" library="SparkFun-Connectors" deviceset="CONN_03" device="JST-PTH"/>
-<part name="J14" library="SparkFun-Connectors" deviceset="CONN_02" device=""/>
-<part name="GND4" library="SparkFun-PowerSymbols" deviceset="GND" device=""/>
 </parts>
 <sheets>
@@
 <instance part="J2" gate="G$1" x="114.3" y="93.98"/>
 <instance part="S_MODE" gate="1" x="185.42" y="104.14"/>
+<instance part="GPSCONN" gate="J$1" x="195.58" y="119.38" rot="R180"/>
 <instance part="X1" gate="G1" x="43.18" y="129.54"/>
 <instance part="LS1" gate="G$1" x="71.12" y="73.66"/>
-<instance part="Q1" gate="G$1" x="83.82" y="66.04" rot="R270"/>
+<instance part="Q1" gate="G$1" x="83.82" y="66.04" rot="R90"/>
 <instance part="S_ANT" gate="1" x="66.04" y="132.08" rot="R180"/>
 <instance part="ANT_EXT" gate="G$1" x="50.8" y="144.78"/>
@@
 <instance part="J11" gate="G$1" x="139.7" y="101.6" rot="R180"/>
 <instance part="J12" gate="G$1" x="121.92" y="116.84" rot="R270"/>
-<instance part="J13" gate="J$1" x="195.58" y="119.38" rot="R180"/>
-<instance part="J14" gate="G$1" x="73.66" y="106.68" rot="R270"/>
-<instance part="GND4" gate="1" x="91.44" y="60.96"/>
 </instances>
 <busses>
@@
 <wire x1="109.22" y1="93.98" x2="109.22" y2="88.9" width="0.1524" layer="91"/>
 <wire x1="132.08" y1="88.9" x2="109.22" y2="88.9" width="0.1524" layer="91"/>
+<pinref part="Q1" gate="G$1" pin="C"/>
+<wire x1="88.9" y1="68.58" x2="101.6" y2="81.28" width="0.1524" layer="91"/>
+<wire x1="101.6" y1="81.28" x2="101.6" y2="88.9" width="0.1524" layer="91"/>
 <pinref part="J5" gate="G$1" pin="1"/>
 <junction x="99.06" y="88.9"/>
@@
 </segment>
 <segment>
+<pinref part="GPSCONN" gate="J$1" pin="1"/>
+<wire x1="187.96" y1="121.92" x2="185.42" y2="121.92" width="0.1524" layer="91"/>
+</segment>
+<segment>
 <pinref part="S_MODE" gate="1" pin="O"/>
 <wire x1="190.5" y1="106.68" x2="193.04" y2="106.68" width="0.1524" layer="91"/>
@@
 <wire x1="129.54" y1="96.52" x2="127" y2="96.52" width="0.1524" layer="91"/>
 </segment>
-<segment>
-<pinref part="J13" gate="J$1" pin="1"/>
-<wire x1="187.96" y1="121.92" x2="185.42" y2="121.92" width="0.1524" layer="91"/>
-</segment>
 </net>
 <net name="NSS" class="0">
@@
 <net name="8" class="0">
 <segment>
+<pinref part="GPSCONN" gate="J$1" pin="3"/>
 <wire x1="187.96" y1="116.84" x2="177.8" y2="106.68" width="0.1524" layer="91"/>
 <wire x1="177.8" y1="106.68" x2="154.94" y2="106.68" width="0.1524" layer="91"/>
@@
 </segment>
 </net>
+<net name="7" class="0">
+<segment>
+<pinref part="S_MODE" gate="1" pin="P"/>
+<wire x1="182.88" y1="104.14" x2="154.94" y2="104.14" width="0.1524" layer="91"/>
+</segment>
+<segment>
+<pinref part="J3" gate="G$1" pin="7"/>
+<wire x1="162.56" y1="104.14" x2="165.1" y2="104.14" width="0.1524" layer="91"/>
+</segment>
+</net>
 <net name="N$3" class="0">
 <segment>
 <pinref part="LS1" gate="G$1" pin="2"/>
-<pinref part="Q1" gate="G$1" pin="C"/>
-<wire x1="78.74" y1="63.5" x2="78.74" y2="66.04" width="0.1524" layer="91"/>
-<wire x1="78.74" y1="66.04" x2="73.66" y2="71.12" width="0.1524" layer="91"/>
+<pinref part="Q1" gate="G$1" pin="E"/>
+<wire x1="73.66" y1="71.12" x2="76.2" y2="68.58" width="0.1524" layer="91"/>
+<wire x1="76.2" y1="68.58" x2="78.74" y2="68.58" width="0.1524" layer="91"/>
 </segment>
 </net>
@@
 </segment>
 <segment>
+<pinref part="GPSCONN" gate="J$1" pin="2"/>
+<wire x1="187.96" y1="119.38" x2="185.42" y2="119.38" width="0.1524" layer="91"/>
+</segment>
+<segment>
 <pinref part="J9" gate="G$1" pin="1"/>
 <wire x1="73.66" y1="134.62" x2="71.12" y2="134.62" width="0.1524" layer="91"/>
@@
 <wire x1="99.06" y1="132.08" x2="101.6" y2="132.08" width="0.1524" layer="91"/>
 </segment>
-<segment>
-<pinref part="J13" gate="J$1" pin="2"/>
-<wire x1="187.96" y1="119.38" x2="185.42" y2="119.38" width="0.1524" layer="91"/>
-</segment>
-<segment>
-<pinref part="J14" gate="G$1" pin="1"/>
-<wire x1="73.66" y1="99.06" x2="73.66" y2="96.52" width="0.1524" layer="91"/>
-</segment>
-<segment>
-<pinref part="Q1" gate="G$1" pin="E"/>
-<wire x1="88.9" y1="63.5" x2="91.44" y2="63.5" width="0.1524" layer="91"/>
-<pinref part="GND4" gate="1" pin="GND"/>
-</segment>
-</net>
-<net name="N$9" class="0">
-<segment>
-<pinref part="J14" gate="G$1" pin="2"/>
-<wire x1="76.2" y1="99.06" x2="76.2" y2="88.9" width="0.1524" layer="91"/>
-</segment>
 </net>
 <net name="N$1" class="0">
 <segment>
 <pinref part="R1" gate="G$1" pin="1"/>
-<wire x1="101.6" y1="60.96" x2="93.98" y2="68.58" width="0.1524" layer="91"/>
 <pinref part="Q1" gate="G$1" pin="B"/>
-<wire x1="93.98" y1="68.58" x2="83.82" y2="68.58" width="0.1524" layer="91"/>
-</segment>
-</net>
-<net name="N$6" class="0">
-<segment>
-<pinref part="J3" gate="G$1" pin="7"/>
-<pinref part="S_MODE" gate="1" pin="P"/>
-<wire x1="162.56" y1="104.14" x2="182.88" y2="104.14" width="0.1524" layer="91"/>
-</segment>
-</net>
+<wire x1="101.6" y1="60.96" x2="83.82" y2="60.96" width="0.1524" layer="91"/>
+<wire x1="83.82" y1="60.96" x2="83.82" y2="63.5" width="0.1524" layer="91"/>
+</segment>
+</net>
